File: kicad-circuits/summer/2-input-summer-inverting.kicad_sch (KiCad schematic)
At the start: 4 parts

Commit message: Reorganized circuits.
Parts:
- R1, R2, R3: value 10k -> (none)
- U1: value (none) -> ~
Changed lines of the file:
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@@
     (in_bom yes) (on_board yes) (fields_autoplaced)
     (property "Reference" "R3" (id 0) (at 118.11 106.68 90))
-    (property "Value" "10k" (id 1) (at 118.11 109.22 90))
+    (property "Value" "" (id 1) (at 118.11 109.22 90))
     (property "Footprint" "" (id 2) (at 118.11 114.808 90)
       (effects (font (size 1.27 1.27)) hide)
@@
     (in_bom yes) (on_board yes)
     (property "Reference" "R1" (id 0) (at 102.87 97.79 90))
-    (property "Value" "10k" (id 1) (at 102.87 100.33 90))
+    (property "Value" "" (id 1) (at 102.87 100.33 90))
     (property "Footprint" "" (id 2) (at 102.87 93.472 90)
       (effects (font (size 1.27 1.27)) hide)
@@
     (in_bom yes) (on_board yes) (fields_autoplaced)
     (property "Reference" "U1" (id 0) (at 129.54 88.011 0))
-    (property "Value" "" (id 1) (at 129.54 90.551 0))
+    (property "Value" "~" (id 1) (at 129.54 90.551 0))
     (property "Footprint" "" (id 2) (at 119.38 92.71 0)
       (effects (font (size 1.27 1.27)) hide)
@@
     (in_bom yes) (on_board yes)
     (property "Reference" "R2" (id 0) (at 102.87 107.95 90))
-    (property "Value" "10k" (id 1) (at 102.87 110.49 90))
+    (property "Value" "" (id 1) (at 102.87 110.49 90))
     (property "Footprint" "" (id 2) (at 102.87 107.188 90)
       (effects (font (size 1.27 1.27)) hide)

Commit message: Updated README and organization of test circuit.
Parts:
- U1: value ~ -> (none); Spice_Lib_File ../../../spice-models/LM358-onsemi.mod -> ../../spice-models/LM358-onsemi.mod
Changed lines of the file:
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@@
     (in_bom yes) (on_board yes) (fields_autoplaced)
     (property "Reference" "U1" (id 0) (at 129.54 88.011 0))
-    (property "Value" "~" (id 1) (at 129.54 90.551 0))
+    (property "Value" "" (id 1) (at 129.54 90.551 0))
     (property "Footprint" "" (id 2) (at 119.38 92.71 0)
       (effects (font (size 1.27 1.27)) hide)
@@
       (effects (font (size 1.27 1.27)) hide)
     )
-    (property "Spice_Lib_File" "../../../spice-models/LM358-onsemi.mod" (id 8) (at 119.38 92.71 0)
+    (property "Spice_Lib_File" "../../spice-models/LM358-onsemi.mod" (id 8) (at 119.38 92.71 0)
       (effects (font (size 1.27 1.27)) hide)
     )
